File: pepper.kicad_sch (KiCad schematic)
At the start: 50 parts, among them J1 USB, J2 Debug, J3 Conn_01x06, Q1 BSS138, SW1 Reset, SW2 Boot, SW3 Action, SW4 Action, U1 ESP32-S3-WROOM-1, U2 AP2112K-3.3

Commit message: Simple order 1
Parts:
- added SW5, SW6: Action, Button_Switch_SMD:SW_SPST_TL3342, symbol Switch:SW_Push
- SW3, SW4: footprint Button_Switch_SMD:SW_SPST_B3U-1000P -> Button_Switch_SMD:SW_SPST_TL3342
Connections:
- net GND: now also SW5.1, SW6.1
- net ESP_IO47: now reaches U1.24 (IO47)
- net ESP_IO47: now also SW5.2
- net ESP_IO48: now reaches U1.25 (IO48)
- net ESP_IO48: now also SW6.2
- no-connect marks 21 -> 19
